File: RFSoC_Frontend_v0.1/RFSoC_Frontend_v0.1.kicad_pcb (KiCad board)
At the start: 4 copper layers, 242.3 x 70.5 mm, 130 parts, among them J1 Conn_Coaxial, J10 LPAM-40-01.0-X-08-X-K-TR, J13 Conn_Coaxial, J14 Conn_Coaxial, J15 Conn_Coaxial, J16 Conn_Coaxial, J17 Conn_Coaxial, J18 Conn_Coaxial, J19 Conn_Coaxial, J2 Conn_Coaxial, J20 Conn_Coaxial, J3 Conn_Coaxial, J4 Conn_Coaxial, J5 Conn_Coaxial, J6 Conn_Coaxial, J7 Conn_Coaxial, J8 Conn_Coaxial, J9 LPAM-40-01.0-X-08-X-K-TR, U1 TCM2-33WX+, U10 TCM2-33WX+, U11 TCM2-33WX+, U12 TCM2-33WX+, U13 TCM2-33WX+, U14 TCM2-33WX+, U15 TCM2-33WX+, U16 TCM2-33WX+, U2 TCM2-33WX+, U3 TCM2-33WX+, U4 TCM2-33WX+, U5 TCM2-33WX+, U6 TCM2-33WX+, U7 TCM2-33WX+, U8 TCM2-33WX+, U9 TCM2-33WX+

Commit message: Transferred Files from Erics Folder
Parts:
- removed C17, C18, C19, C20, C21, C22, C23, C24, C25, C26, C27, C28, C29, C30, C31, C32: .01u, Capacitor_SMD:C_0402_1005Metric
- removed J13, J14, J15, J16, J17, J18, J19, J20: Conn_Coaxial, Connector_Coaxial:SMA_Amphenol_132289_EdgeMount
- removed R33, R34, R35, R36, R45, R46, R47, R48, R49, R50, R51, R52, R61, R62, R63, R64: 590, Resistor_SMD:R_0402_1005Metric
- removed R37, R38, R39, R40, R41, R42, R43, R44, R53, R54, R55, R56, R57, R58, R59, R60: 17.4, Resistor_SMD:R_0402_1005Metric
- removed U10, U11, U12, U13, U14, U15, U16, U9: TCM2-33WX+, MINICIRCUITS:XFMR_TCM2-33WX+
- added REF: MountingHole_2.2mm_M2_DIN965_Pad, MountingHole:MountingHole_2.2mm_M2_DIN965_Pad, F.Cu at (68.6, 0.00)
- added REF: MountingHole_2.2mm_M2_DIN965_Pad, MountingHole:MountingHole_2.2mm_M2_DIN965_Pad, F.Cu at (-6.43, 0.00)
- added e: MountingHole_2.2mm_M2_DIN965_Pad, MountingHole:MountingHole_2.2mm_M2_DIN965_Pad, F.Cu at (143.6, 0.00)
- J1, J2, J3, J4, J5, J6, J7, J8: footprint Connector_Coaxial:SMA_Amphenol_132289_EdgeMount -> local:SMA_Amphenol_132289_EdgeMount
- J10, J9: footprint LPAM:SAMTEC_LPAM-40-01.0-X-08-X-K-TR -> local:SAMTEC_LPAM-40-01.0-X-08-X-K-TR
- U1, U2, U3, U4, U5, U6, U7, U8: footprint MINICIRCUITS:XFMR_TCM2-33WX+ -> local:XFMR_TCM2-33WX+
- moved J3 169.4 mm to (81.3, 23.8)
- moved C6 168.9 mm to (78.1, 14.0)
- moved R3 168.3 mm to (79.7, 8.00)
- moved R10 168.3 mm to (79.2, 9.78)
- moved R9 168.3 mm to (80.2, 9.78)
- moved R15 168.3 mm to (79.7, 11.6)
- moved U3 168.1 mm to (79.7, 17.4)
- moved C5 167.1 mm to (81.3, 14.0)
- moved J1 141.9 mm to (127.0, 23.8)
- moved C2 141.1 mm to (123.8, 14.0)
- moved R13 140.6 mm to (125.4, 11.6)
- moved R1 140.6 mm to (125.4, 8.00)
- moved R6 140.6 mm to (124.9, 9.78)
- moved R5 140.6 mm to (125.9, 9.78)
- moved U1 140.3 mm to (125.4, 17.4)
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Routing:
- net GND: track 0.00 -> 106.7 mm, vias 3 -> 64
- net ADC_B0_N: track 3.71 -> 45.9 mm, vias 2 -> 1
- net ADC_B0_P: track 4.09 -> 44.0 mm, vias 2 -> 1
- net DAC_A1_N: track 3.12 -> 32.1 mm, vias 2 -> 1
- net DAC_A1_P: track 3.50 -> 30.1 mm, vias 2 -> 1
- net ADC_A0_N: track 3.19 -> 25.6 mm
- net ADC_A0_P: track 3.19 -> 23.7 mm
- net ADC_B1_N: track 7.31 -> 26.7 mm, vias 2 -> 1
- net ADC_A1_N: track 3.74 -> 22.0 mm
- net DAC_B1_N: track 9.50 -> 27.6 mm, vias 2 -> 1
- net ADC_B1_P: track 7.12 -> 24.7 mm, vias 2 -> 1
- net ADC_A1_P: track 2.47 -> 20.1 mm
- net DAC_B1_P: track 9.62 -> 25.7 mm, vias 2 -> 1
- net DAC_A0_N: track 3.56 -> 15.9 mm, vias 2 -> 1
- net DAC_A0_P: track 3.37 -> 13.9 mm, vias 2 -> 1
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Other:
- board size 242.3 x 70.5 mm -> 165.1 x 37.1 mm
- net class Default removed
- board text added: "Notes : Check Breakout Mounting Hole screw sizes"

Commit message: added labels
Parts:
- moved C10 110.8 mm to (109.9, 97.8)
- moved C11 110.8 mm to (82.6, 97.8)
- moved C12 110.8 mm to (79.5, 97.8)
- moved C13 110.8 mm to (97.9, 97.8)
- moved C15 110.8 mm to (128.3, 97.8)
- moved C16 110.8 mm to (125.2, 97.8)
- moved C2 110.8 mm to (196.3, 97.8)
- moved C3 110.8 mm to (184.2, 97.8)
- moved C4 110.8 mm to (181.1, 97.8)
- moved C6 110.8 mm to (150.6, 97.8)
- moved C7 110.8 mm to (169.0, 97.8)
- moved C8 110.8 mm to (165.8, 97.8)
- moved C9 110.8 mm to (113.1, 97.8)
- moved J2 110.8 mm to (184.2, 107.7)
- moved J4 110.8 mm to (169.0, 107.7)
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Other:
- board text added: "1"
- board text added: "10"
- board text added: "15"
- board text added: "20"
- board text added: "25"
- board text added: "30"
- board text added: "35"
- board text added: "40"
- board text added: "5"
- board text added: "A"
- board text added: "B"
- board text added: "B19"
- board text added: "B19,C19 RFMC_DAC_06"
- board text added: "C"
- board text added: "C19"
- board text added: "D"
- board text added: "E"
- board text added: "F"
- board text added: "F20"
- board text added: "F20,G20 RFMC_ADC_07"
- board text added: "G"
- board text added: "G20"
- board text added: "H"
- board text added: "RFMC ADC"
- board text added: "RFMC DAC"
